File: Clock_board.kicad_pcb (KiCad board)
At the start: 2 copper layers, 70 x 70 mm, 34 parts, among them J1 Conn_01x02, J2 Conn_01x02, J3 Conn_01x02, J4 Conn_01x02, J5 Conn_01x02, SW1 SW_Push, SW2 SW_Push_DPDT, U1 NE555, U2 NE555, U3 NE555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

Commit message: Fixed the resistor footprints and changed revision to B
Parts:
- R1, R2, R3, R4, R5, R6: footprint Resistor_THT:R_Axial_DIN0204_L3.6mm_D1.6mm_P5.08mm_Horizontal -> Resistor_THT:R_Axial_DIN0207_L6.3mm_D2.5mm_P7.62mm_Horizontal
- moved C5 3.81 mm to (143.5, 64.8)
- moved R2 1.27 mm to (127.0, 73.7)
- moved R5 1.27 mm to (143.5, 74.9)
- moved R6 1.27 mm to (121.9, 73.7)
Routing:
- net +5V: track 130.6 -> 133.8 mm, vias 0 -> 1
- net Net-(R6-Pad1): track 21.1 -> 19.9 mm
- net /DISCH_1: track 11.4 -> 10.3 mm
- net /TRIG_3: track 17.0 -> 18.2 mm
- net /THRES_2: track 10.2 -> 10.7 mm
- net /TRIG_2: track 24.6 -> 25.2 mm
Other:
- board text added: "Rev: B"
- board text removed: "Rev: A"
